Commit message: added modified lidar positions

File: urdf/m20_with_arm/m20_with_arm.urdf (robot description, URDF)
Before this commit: robot M20, 18 links, 18 joints
Links:
- added link camera_front_link, mass 0.072; collision box size=0.040 0.090 0.025; visual box size=0.040 0.090 0.025
- added link camera_rear_link, mass 0.072; collision box size=0.040 0.090 0.025; visual box size=0.040 0.090 0.025
- added link imu_link, mass 0.015; collision box size=0.020 0.020 0.010; visual box size=0.020 0.020 0.010
- added link lidar_front_link, mass 0.190; collision cylinder length=0.040 radius=0.035; visual cylinder length=0.040 radius=0.035
- added link lidar_rear_link, mass 0.190; collision cylinder length=0.040 radius=0.035; visual cylinder length=0.040 radius=0.035
Joints:
- added joint camera_front_joint: type fixed, parent base_link, child camera_front_link, origin xyz=0.37646 0.0 0.03738 rpy=0 0 0
- added joint camera_rear_joint: type fixed, parent base_link, child camera_rear_link, origin xyz=-0.37646 0.0 0.03738 rpy=0 0 3.14159265
- added joint imu_joint: type fixed, parent base_link, child imu_link, origin xyz=0.0632 -0.0268 -0.0435 rpy=0 0 0
- added joint lidar_front_joint: type fixed, parent base_link, child lidar_front_link, origin xyz=0.43 0.0 0.11 rpy=0 0 0
- added joint lidar_rear_joint: type fixed, parent base_link, child lidar_rear_link, origin xyz=-0.43 0.0 0.11 rpy=0 0 3.14159265
